Commit message: * Corrected robot model. * Added amcl demo. * Reorganized repo. * Added example map. * Updated readme.

File: robots/kobuki_hexagons_rplidar.urdf.xacro (robot description, xacro)
@@ -9,5 +9,5 @@
     <xacro:include filename="$(find kobuki_description)/urdf/kobuki.urdf.xacro" />
     <xacro:include filename="$(find turtlebot_description)/urdf/stacks/hexagons.urdf.xacro"/>
-    <xacro:include filename="$(find mapping_with_lidar)/urdf/rplidar.urdf.xacro"/>
+    <xacro:include filename="$(find turtlebot_with_lidar)/urdf/rplidar.urdf.xacro"/>
     <kobuki/>
     <stack_hexagons parent="base_link"/>

File: urdf/rplidar.urdf.xacro (robot description, xacro)
@@ -5,5 +5,5 @@
     <xacro:macro name="sensor_rplidar" params="parent">
     <joint name="laser" type="fixed">
-        <origin xyz="0.180 0.00 0.040" rpy="0 0 0" />
+        <origin xyz="0.180 0.00 0.040" rpy="3.1416 0 0" />
         <parent link="${parent}" />
         <child link="base_laser_link" />
@@ -13,5 +13,5 @@
             <origin xyz="-0.0425 0.035 -0.040" rpy="1.570796327 0 0"/>
             <geometry>
-                <mesh filename="package://mapping_with_lidar/meshes/rplidar_main.STL" scale="0.001 0.001 0.001"/>
+                <mesh filename="package://turtlebot_with_lidar/meshes/rplidar_main.STL" scale="0.001 0.001 0.001"/>
             </geometry>
             <material name="blue">
